File: interacto.brd (EAGLE design)
At the start: 101.4 x 57.3 mm, 87 parts

Commit message: BOM done.
Parts:
- LED1: value (none) -> blue
- LED2, LED3: value (none) -> green
- R10, R11, R12, R13, R14, R15, R16, R17, R18, R19, R20, R21, R22, R23, R24, R25, R26, R27, R28, R29, R30, R31, R37, R38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: value (none) -> 33
- R33: value 4.75K -> 150
- R34, R35: value 4.75K -> 50
- R36: value (none) -> 10K
