File: interacto.sch (EAGLE design)
At the start: 87 parts

Commit message: BOM done.
Parts:
- C1, C10, C14, C15, C2, C23, C24, C25, C26, C27, C28, C3, C6, C9: MPN (none) -> VJ0603V104ZXXCW1BC
- C11, C7: MPN (none) -> VJ0603V224MXJPW1BC
- C12, C5: MPN (none) -> GRM188F51A475ZE20J
- C13, C4, C8: MPN (none) -> LMK107BBJ106MALT
- C16, C18, C21: MPN (none) -> VJ0603Y103KXACW1BC
- C17, C19, C20: MPN (none) -> C1608X7R1C105K
- C22: MPN (none) -> C1608Y5V1C225Z
- LED1: value (none) -> blue; MPN (none) -> HT-193NB-5589
- LED2, LED3: value (none) -> green; MPN (none) -> LG Q971-KN-1
- P6: MPN (none) -> SSHQ-105-D-10-GT-LF
- P8, P9: MPN (none) -> SSHQ-123-D-10-GT-LF
- R1, R3: MPN (none) -> RK73B1JTTDD562J
- R10, R11, R12, R13, R14, R15, R16, R17, R18, R19, R20, R21, R22, R23, R25, R26, R27, R28, R29, R30, R31, R37, R38, R6, R8: value (none) -> 33; MPN (none) -> CR0402-JW-330GLF
- R2, R4, R5, R7: MPN (none) -> CR0603-FX-4751GLF
- R24: value (none) -> 33
- R32, R9: MPN (none) -> WR06X1002FTL
- R33: value 4.75K -> 150; MPN (none) -> 302-150-RC
- R34, R35: value 4.75K -> 50; MPN (none) -> 302-49.9-RC
- R36: value (none) -> 10K; MPN (none) -> WR06X1002FTL
- S1: MPN (none) -> 219-2MST
- U$1: MPN (none) -> CAT24C256WI-GT3
- U$10: MPN (none) -> LP3985IM5-2.8/NOPB
- U$12: MPN (none) -> TPS79915DDCR
- U$13: MPN (none) -> SN74LVCH16T245DGGR
- U$3: MPN (none) -> TCM8230MD
- U$4: MPN (none) -> SN74LVC1T45DBVR
- U$5: MPN (none) -> LSM303DLHC
- U$7: MPN (none) -> LSM330DLC
- U$8: MPN (none) -> LSM333D
Other:
- note added: "Interacto"
- note removed: "Cape Name"
