File: Hardware/interacto.brd (EAGLE design)
At the start: 101.4 x 57.3 mm, 87 parts

Commit message: Updates from prototype build and testing.
Parts:
- removed R30: 33, rcl:R0402
- C10, C9: value 0.1u -> 0.1u, DNI
- C11: value 0.22u -> 0.22u, DNI
- C12: value 4.7u -> 4.7u, DNI
- C8: value 10u -> 10u, DNI
- R10, R11, R12, R13, R14, R15, R16, R17, R18, R19, R20, R21, R22, R23, R24, R25, R26, R27, R28, R29, R37, R38, R6, R8: value 33 -> 100
- R31: value 33 -> 0
- R32: value 10K -> 100
- R36: value 10K -> 50
- U$8: value (none) -> DNI
Connections:
- removed net N$22: R18.1, U$13.16
- removed net N$41: R30.2, U$13.33
- net GPIO2_24: now also R18.1; no longer R30.1
Routing:
- net GPIO2_24: track 42.8 -> 99.0 mm
- net N$41: track 9.66 -> 0.00 mm
- net N$22: track 9.14 -> 0.00 mm
