File: Hardware/interacto.sch (EAGLE design)
At the start: 87 parts

Commit message: Updates from prototype build and testing.
Parts:
- removed R30: 33, rcl:R-US_R0402
- C10, C9: value 0.1u -> 0.1u, DNI
- C11: value 0.22u -> 0.22u, DNI
- C12: value 4.7u -> 4.7u, DNI
- C8: value 10u -> 10u, DNI
- R10, R11, R12, R13, R14, R15, R16, R17, R18, R19, R20, R21, R22, R23, R25, R26, R28, R29, R37, R38, R6, R8: value 33 -> 100; MPN CR0402-JW-330GLF -> ERA-6AED101V
- R24: value 33 -> 100; MPN (none) -> ERA-6AED101V
- R27: value 33 -> 100
- R31: value 33 -> 0; MPN CR0402-JW-330GLF -> ERJ-2GE0R00X
- R32: value 10K -> 100; MPN WR06X1002FTL -> ERA-6AED101V
- R36: value 10K -> 50; MPN WR06X1002FTL -> 302-49.9-RC
- U$8: value (none) -> DNI
Connections:
- removed net N$22: R18.1, U$13.2B3
- removed net N$41: R30.2, U$13.2A3
- net GPIO2_24: now also R18.1; no longer R30.1
